File: pcb/LiPoBCB.kicad_pcb (KiCad board)
At the start: 2 copper layers, 30 x 16.5 mm, 27 parts, among them J1 USB-C_6_pin_receptacle, J2 Conn_01x02, Q1 Q_Dual_PMOS_S1G1D2S2G2D1, U1 ETA9740

Commit message: Update pcb files
Parts:
- moved R7 13.3 mm to (146.7, 64.5), turned to -90 degrees
- moved R4 12.8 mm to (152.4, 52.3)
- moved R5 12.7 mm to (150.6, 52.3)
- moved C6 12.2 mm to (148.2, 64.5), turned to -90 degrees
- moved TP1 1.28 mm to (140.9, 51.6)
- moved TP2 1.28 mm to (137.3, 51.6)
- moved C2 0.41 mm to (143.5, 64.5)
- moved R1 0.41 mm to (145.0, 64.5)
- moved C3 0.40 mm to (146.5, 59.6)
- moved C4 0.40 mm to (142.7, 58.2)
- moved D2 0.40 mm to (133.5, 60.1)
- moved D4 0.40 mm to (133.5, 63.2)
- moved J2 0.40 mm to (150.9, 64.5)
- moved L1 0.40 mm to (138.5, 57.3)
- moved R3 0.40 mm to (133.4, 64.7)
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Connections:
- Q1 pad 4: +5V -> /VBUS
- Q1 pad 6: /VBUS -> +5V
Routing:
- net Net-(C6-Pad2): track 16.0 -> 4.53 mm, vias 1 -> 0
- net /CC2: track 17.6 -> 9.67 mm
- net /CC1: track 17.3 -> 11.1 mm
- net Net-(C5-Pad1): track 5.67 -> 7.45 mm, vias 0 -> 2
- net /ISET: track 5.77 -> 4.02 mm, vias 2 -> 0
- net /SW_GATE: track 13.9 -> 12.7 mm, vias 2 -> 0
- net GND: track 1.24 -> 0.37 mm, vias 6 -> 12
- net /VBUS: track 0.36 -> 0.00 mm, vias 4 -> 6
- net /BAT: track 0.35 -> 0.02 mm, vias 7 -> 8

Commit message: Updates DRC
Parts:
- removed TP1: 5V, TestPoint:TestPoint_THTPad_2.5x2.5mm_Drill1.2mm
- removed TP2: GND, TestPoint:TestPoint_THTPad_2.5x2.5mm_Drill1.2mm
- added P1: Solder_Connector_X2, LiPoBCB-V2:Solder_Connector_X2, F.Cu at (140.3, 51.5)
- J2: footprint Connector_PinHeader_2.54mm:PinHeader_1x02_P2.54mm_Vertical -> LiPoBCB-V2:Solder_Connector_SW
- moved J2 0.62 mm to (150.9, 65.2), turned to 0 degrees
- moved C5 0.13 mm to (151.1, 60.1)
- moved R6 0.13 mm to (152.7, 60.1)
- moved J1 0.06 mm to (154.7, 56.1)
Routing:
- net GND: vias 12 -> 14
- net /BAT: vias 8 -> 7
Other:
- board text added: "LiPoBCB V2.0 Jakob Holz - 03.12.22"
- board text added: "max.2A"
- board text added: "on/off"
